Commit message: Added Inertial tags to URDF

File: arthrobot_ws/src/arthrobot_description/urdf/arthrobot.urdf.xacro (robot description, xacro)
@@ -1,4 +1,18 @@
 <?xml version="1.0"?>
-<robot name = "arthrobot">
+<robot xmlns:xacro="http://www.ros.org/wiki/xacro" name="arthrobot">
+    <!-- Useful XACRO Variables (Properties) -->
+    <xacro:property name="PI" value="3.14159265359" />
+    <xacro:property name="effort" value="30.0" />
+    <xacro:property name="velocity" value="10.0" />
+    <!-- Useful Macros -->
+    <xacro:macro name="default_inertial" params="mass">
+        <inertial>
+            <origin xyz="0 0 0" rpy="0 0 0"/>
+            <mass value="${mass}" />
+            <inertia ixx="1.0" ixy="0.0" ixz="0.0"
+                     iyy="1.0" iyz="0.0"
+                     izz="1.0" />
+        </inertial>
+    </xacro:macro>
 <!-- This is the first link: empty link specifying the world -->
 <link name="world"></link>
@@ -11,4 +25,5 @@
 <!-- The base link (wooden frame and the metalic support)-->
 <link name="base_link">
+    <xacro:default_inertial mass="5.0"/>
     <visual>
         <origin xyz="0.0 0.0 0.0225" rpy="0.0 0.0 0.0"/>
@@ -50,4 +65,5 @@
 <!--Motor 1 link-->
 <link name="motor1_link">
+    <xacro:default_inertial mass="0.1"/>
     <visual>
         <origin xyz="0.0 0.0 0.005" rpy="0.0 0.0 0.0"/>
@@ -91,4 +107,5 @@
 <!--Motor 2 link-->
 <link name="motor2_link">
+    <xacro:default_inertial mass="0.1"/>
     <visual>
         <origin xyz="0.0 0.01 0.0125" rpy="0.0 0.0 0.0"/>
@@ -117,4 +134,5 @@
 <!--bar 1 link-->
 <link name="bar1_link">
+    <xacro:default_inertial mass="0.1"/>
     <visual>
         <origin xyz="-0.001 0.0 0.0525" rpy="0.0 0.0 0.0"/>
@@ -158,4 +176,5 @@
 <!--bar 2 link-->
 <link name="bar2_link">
+    <xacro:default_inertial mass="0.1"/>
     <visual>
         <origin xyz="-0.001 0.0 0.049" rpy="0.0 0.0 0.0"/>
@@ -199,4 +218,5 @@
 <!--motor 3 link-->
 <link name="motor3_link">
+    <xacro:default_inertial mass="0.1"/>
     <visual>
         <origin xyz="0.0285 0.01 0.0" rpy="0.0 0.0 0.0"/>
@@ -223,4 +243,5 @@
 <!-- motor 4 link-->
 <link name="motor4_link">
+    <xacro:default_inertial mass="0.1"/>
     <visual>
         <origin xyz="0.0 0.0 0.023" rpy="0.0 0.0 0.0"/>
@@ -249,4 +270,5 @@
 <!-- ee link (end effector)-->
 <link name="ee_link">
+    <xacro:default_inertial mass="0.05"/>
     <visual>
         <origin xyz="0.0 0.0 0.012" rpy="-1.57 0.0 0.0"/>

Commit message: Added Control Tags to URDF

File: arthrobot_ws/src/arthrobot_description/urdf/arthrobot.urdf.xacro (robot description, xacro)
@@ -1,4 +1,6 @@
 <?xml version="1.0"?>
 <robot xmlns:xacro="http://www.ros.org/wiki/xacro" name="arthrobot">
+    <!-- Include Gazebo Parameters -->
+    <xacro:include filename="$(find arthrobot_description)/urdf/arthrobot_gazebo.xacro" />
     <!-- Useful XACRO Variables (Properties) -->
     <xacro:property name="PI" value="3.14159265359" />
@@ -15,4 +17,13 @@
         </inertial>
     </xacro:macro>
+    <xacro:macro name="default_transmission" params="number">
+        <transmission name="transmission_${number}">
+            <plugin>transmission_interface/SimpleTransmission</plugin>
+            <actuator name="motor_${number}" role="actuator1"/>
+            <joint name="joint_${number}"    role="joint1">
+                <mechanical_reduction>1.0</mechanical_reduction>
+            </joint>
+        </transmission>
+    </xacro:macro>
 <!-- This is the first link: empty link specifying the world -->
 <link name="world"></link>
@@ -58,5 +69,5 @@
 </link>
 <!-- Joint that attaches the base with motor 1-->
-<joint name="base_motor1_joint" type="fixed">
+<joint name="base_motor_link" type="fixed">
     <origin xyz="-0.007 0.0085 0.081" rpy="0.0 0.0 0.0"/>
     <parent link="base_link"/>
@@ -98,5 +109,5 @@
 </link>
 <!--Joint between motor 1 and motor 2-->
-<joint name="motor1_motor2_joint" type="revolute">
+<joint name="joint_1" type="revolute">
     <origin xyz="-0.01 0.0 0.018" rpy="0.0 0.0 0.0"/>
     <parent link="motor1_link"/>
@@ -125,5 +136,5 @@
 </link>
 <!--Joint between motor 2 and bar 1-->
-<joint name="motor2_bar1_joint" type="revolute">
+<joint name="joint_2" type="revolute">
     <origin xyz="-0.0285 0.02 0.0125" rpy="0.0 0.0 0.0"/>
     <parent link="motor2_link"/>
@@ -167,5 +178,5 @@
 </link>
 <!--joint between bar 1 and bar 2-->
-<joint name="bar1_bar2_joint" type="revolute">
+<joint name="joint_3" type="revolute">
     <origin xyz="-0.002 0.0 0.105" rpy="0.0 0.0 0.0"/>
     <parent link="bar1_link"/>
@@ -209,5 +220,5 @@
 </link>
 <!--joint bar 2 motor 3-->
-<joint name="bar2_motor3_joint" type="revolute">
+<joint name="joint_4" type="revolute">
     <origin xyz="0.002 0.0 0.098" rpy="0.0 0.0 0.0"/>
     <parent link="bar2_link"/>
@@ -261,5 +272,5 @@
 </link>
 <!--Joint motor 4 ee link-->
-<joint name="motor4_ee_joint" type="revolute">
+<joint name="joint_5" type="revolute">
     <origin xyz="-0.01 0.0 0.046" rpy="0.0 0.0 0.0"/>
     <parent link="motor4_link"/>
@@ -287,3 +298,9 @@
     </collision>
 </link>
+<!-- Transmissions-->
+<xacro:default_transmission number="1"/>
+<xacro:default_transmission number="2"/>
+<xacro:default_transmission number="3"/>
+<xacro:default_transmission number="4"/>
+<xacro:default_transmission number="5"/>
 </robot>

Commit message: Removed unnecessary files and code for later editing

File: arthrobot_ws/src/arthrobot_description/urdf/arthrobot.urdf.xacro (robot description, xacro)
@@ -1,6 +1,4 @@
 <?xml version="1.0"?>
 <robot xmlns:xacro="http://www.ros.org/wiki/xacro" name="arthrobot">
-    <!-- Include Gazebo Parameters -->
-    <xacro:include filename="$(find arthrobot_description)/urdf/arthrobot_gazebo.xacro" />
     <!-- Useful XACRO Variables (Properties) -->
     <xacro:property name="PI" value="3.14159265359" />
@@ -17,13 +15,4 @@
         </inertial>
     </xacro:macro>
-    <xacro:macro name="default_transmission" params="number">
-        <transmission name="transmission_${number}">
-            <plugin>transmission_interface/SimpleTransmission</plugin>
-            <actuator name="motor_${number}" role="actuator1"/>
-            <joint name="joint_${number}"    role="joint1">
-                <mechanical_reduction>1.0</mechanical_reduction>
-            </joint>
-        </transmission>
-    </xacro:macro>
 <!-- This is the first link: empty link specifying the world -->
 <link name="world"></link>
@@ -42,7 +31,4 @@
             <box size="0.19 0.16 0.045"/>
         </geometry>
-        <material name="wood">
-            <color rgba="0.64 0.454 0.286 1.0"/>
-        </material>
     </visual>
     <collision>
@@ -57,7 +43,4 @@
             <box size="0.07 0.06 0.036"/>
         </geometry>
-        <material name="black">
-            <color rgba="0.0001 0.0001 0.0001 1.0"/>
-        </material>
     </visual>
     <collision>
@@ -82,7 +65,4 @@
             <box size="0.04 0.022 0.01"/>
         </geometry>
-        <material name="red">
-            <color rgba="1.0 0.0 0.0 1.0"/>
-        </material>
     </visual>
     <collision>
@@ -97,7 +77,4 @@
             <cylinder radius="0.006" length="0.008"/>
         </geometry>
-        <material name="white">
-            <color rgba="1.0 1.0 1.0 1.0"/>
-        </material>
     </visual>
     <collision>
@@ -124,7 +101,4 @@
             <box size="0.057 0.06 0.025"/>
         </geometry>
-        <material name="black">
-            <color rgba="0.0 0.0 0.0 1.0"/>
-        </material>
     </visual>
     <collision>
@@ -151,7 +125,4 @@
             <box size="0.002 0.025 0.105"/>
         </geometry>
-        <material name="black">
-            <color rgba="0.09 0.09 0.09 1.0"/>
-        </material>
     </visual>
     <collision>
@@ -166,7 +137,4 @@
             <box size="0.002 0.025 0.105"/>
         </geometry>
-        <material name="black">
-            <color rgba="0.09 0.09 0.09 1.0"/>
-        </material>
     </visual>
     <collision>
@@ -193,7 +161,4 @@
             <box size="0.002 0.025 0.098"/>
         </geometry>
-        <material name="black">
-            <color rgba="0.09 0.09 0.09 1.0"/>
-        </material>
     </visual>
     <collision>
@@ -208,7 +173,4 @@
             <box size="0.002 0.025 0.098"/>
         </geometry>
-        <material name="black">
-            <color rgba="0.09 0.09 0.09 1.0"/>
-        </material>
     </visual>
     <collision>
@@ -235,7 +197,4 @@
             <box size="0.056 0.06 0.025"/>
         </geometry>
-        <material name="black">
-            <color rgba="0.0 0.0 0.0 1.0"/>
-        </material>
     </visual>
     <collision>
@@ -260,7 +219,4 @@
             <box size="0.042 0.022 0.046"/>
         </geometry>
-        <material name="black">
-            <color rgba="0.0 0.0 0.0 1.0"/>
-        </material>
     </visual>
     <collision>
@@ -287,7 +243,4 @@
             <cylinder radius="0.012" length="0.145"/>
         </geometry>
-        <material name="black">
-            <color rgba="1.0 0.0 0.0 1.0"/>
-        </material>
     </visual>
     <collision>
@@ -298,9 +251,3 @@
     </collision>
 </link>
-<!-- Transmissions-->
-<xacro:default_transmission number="1"/>
-<xacro:default_transmission number="2"/>
-<xacro:default_transmission number="3"/>
-<xacro:default_transmission number="4"/>
-<xacro:default_transmission number="5"/>
 </robot>

Commit message: Adjusted effort and velocity parameters of the joints

File: arthrobot_ws/src/arthrobot_description/urdf/arthrobot.urdf.xacro (robot description, xacro)
@@ -3,6 +3,6 @@
     <!-- Useful XACRO Variables (Properties) -->
     <xacro:property name="PI" value="3.14159265359" />
-    <xacro:property name="effort" value="30.0" />
-    <xacro:property name="velocity" value="10.0" />
+    <xacro:property name="effort" value="30.0000000001" />
+    <xacro:property name="velocity" value="10.0000000001" />
     <!-- Useful Macros -->
     <xacro:macro name="default_inertial" params="mass">
@@ -10,6 +10,6 @@
             <origin xyz="0 0 0" rpy="0 0 0"/>
             <mass value="${mass}" />
-            <inertia ixx="1.0" ixy="0.0" ixz="0.0"
-                     iyy="1.0" iyz="0.0"
+            <inertia ixx="1.0" ixy="0.0000000001" ixz="0.0000000001"
+                     iyy="1.0" iyz="0.0000000001"
                      izz="1.0" />
         </inertial>
@@ -19,5 +19,5 @@
 <!--This is the joint that links the robot's base to the world frame -->
 <joint name="world_base_joint" type="fixed">
-    <origin xyz="0.0 0.0 0.0" rpy="0.0 0.0 0.0"/>
+    <origin xyz="0.000000001 0.000000001 0.0000000001" rpy="0.000000001 0.000000001 0.0000000001"/>
     <parent link="world"/>
     <child link="base_link"/>
@@ -25,7 +25,7 @@
 <!-- The base link (wooden frame and the metalic support)-->
 <link name="base_link">
-    <xacro:default_inertial mass="5.0"/>
-    <visual>
-        <origin xyz="0.0 0.0 0.0225" rpy="0.0 0.0 0.0"/>
+    <xacro:default_inertial mass="2.0"/>
+    <visual>
+        <origin xyz="0.000000001 0.000000001 0.0225" rpy="0.000000001 0.000000001 0.0000000001"/>
         <geometry>
             <box size="0.19 0.16 0.045"/>
@@ -33,5 +33,5 @@
     </visual>
     <collision>
-        <origin xyz="0.0 0.0 0.00225" rpy="0.0 0.0 0.0"/>
+        <origin xyz="0.000000001 0.000000001 0.00225" rpy="0.000000001 0.000000001 0.0000000001"/>
         <geometry>
             <box size="0.19 0.16 0.045"/>
@@ -39,5 +39,5 @@
     </collision>
      <visual>
-        <origin xyz="-0.007 0.0085 0.063" rpy="0.0 0.0 0.0"/>
+        <origin xyz="-0.007 0.0085 0.063" rpy="0.000000001 0.000000001 0.0000000001"/>
         <geometry>
             <box size="0.07 0.06 0.036"/>
@@ -45,5 +45,5 @@
     </visual>
     <collision>
-        <origin xyz="-0.007 0.0085 0.063" rpy="0.0 0.0 0.0"/>
+        <origin xyz="-0.007 0.0085 0.063" rpy="0.000000001 0.000000001 0.0000000001"/>
         <geometry>
             <box size="0.07 0.06 0.036"/>
@@ -53,5 +53,5 @@
 <!-- Joint that attaches the base with motor 1-->
 <joint name="base_motor_link" type="fixed">
-    <origin xyz="-0.007 0.0085 0.081" rpy="0.0 0.0 0.0"/>
+    <origin xyz="-0.007 0.0085 0.081" rpy="0.000000001 0.000000001 0.0000000001"/>
     <parent link="base_link"/>
     <child link="motor1_link"/>
@@ -59,7 +59,7 @@
 <!--Motor 1 link-->
 <link name="motor1_link">
-    <xacro:default_inertial mass="0.1"/>
-    <visual>
-        <origin xyz="0.0 0.0 0.005" rpy="0.0 0.0 0.0"/>
+    <xacro:default_inertial mass="0.3"/>
+    <visual>
+        <origin xyz="0.000000001 0.000000001 0.005" rpy="0.000000001 0.000000001 0.0000000001"/>
         <geometry>
             <box size="0.04 0.022 0.01"/>
@@ -67,5 +67,5 @@
     </visual>
     <collision>
-        <origin xyz="0.0 0.0 0.005" rpy="0.0 0.0 0.0"/>
+        <origin xyz="0.000000001 0.000000001 0.005" rpy="0.000000001 0.000000001 0.0000000001"/>
         <geometry>
             <box size="0.04 0.022 0.01"/>
@@ -73,5 +73,5 @@
     </collision>
     <visual>
-        <origin xyz="-0.01 0.0 0.014" rpy="0.0 0.0 0.0"/>
+        <origin xyz="-0.01 0.000000001 0.014" rpy="0.000000001 0.000000001 0.0000000001"/>
         <geometry>
             <cylinder radius="0.006" length="0.008"/>
@@ -79,5 +79,5 @@
     </visual>
     <collision>
-        <origin xyz="-0.01 0.0 0.004" rpy="0.0 0.0 0.0"/>
+        <origin xyz="-0.01 0.000000001 0.004" rpy="0.000000001 0.000000001 0.0000000001"/>
         <geometry>
             <cylinder radius="0.006" length="0.008"/>
@@ -87,15 +87,15 @@
 <!--Joint between motor 1 and motor 2-->
 <joint name="joint_1" type="revolute">
-    <origin xyz="-0.01 0.0 0.018" rpy="0.0 0.0 0.0"/>
+    <origin xyz="-0.01 0.000000001 0.018" rpy="0.000000001 0.000000001 0.0000000001"/>
     <parent link="motor1_link"/>
     <child link="motor2_link"/>
-    <axis xyz="0.0 0.0 1.0"/>
-    <limit lower="-3.1415" upper="3.1415" effort="100" velocity="80"/>
+    <axis xyz="0.000000001 0.000000001 1.0"/>
+    <limit lower="-3.1415" upper="3.1415" effort="80" velocity="50"/>
 </joint>
 <!--Motor 2 link-->
 <link name="motor2_link">
-    <xacro:default_inertial mass="0.1"/>
-    <visual>
-        <origin xyz="0.0 0.01 0.0125" rpy="0.0 0.0 0.0"/>
+    <xacro:default_inertial mass="0.2"/>
+    <visual>
+        <origin xyz="0.000000001 0.01 0.0125" rpy="0.000000001 0.000000001 0.0000000001"/>
         <geometry>
             <box size="0.057 0.06 0.025"/>
@@ -103,5 +103,5 @@
     </visual>
     <collision>
-        <origin xyz="0.0 0.01 0.0125" rpy="0.0 0.0 0.0"/>
+        <origin xyz="0.000000001 0.01 0.0125" rpy="0.000000001 0.000000001 0.0000000001" />
         <geometry>
             <box size="0.057 0.06 0.025"/>
@@ -111,9 +111,9 @@
 <!--Joint between motor 2 and bar 1-->
 <joint name="joint_2" type="revolute">
-    <origin xyz="-0.0285 0.02 0.0125" rpy="0.0 0.0 0.0"/>
+    <origin xyz="-0.0285 0.02 0.0125" rpy="0.000000001 0.000000001 0.0000000001"/>
     <parent link="motor2_link"/>
     <child link="bar1_link"/>
-    <axis xyz="-1.0 0.0 0.0"/>
-    <limit lower="-3.1415" upper="3.1415" effort="100" velocity="80"/>
+    <axis xyz="-1.0 0.000000001 0.0000000001"/>
+    <limit lower="-3.1415" upper="3.1415" effort="80" velocity="50"/>
 </joint>
 <!--bar 1 link-->
@@ -121,23 +121,23 @@
     <xacro:default_inertial mass="0.1"/>
     <visual>
-        <origin xyz="-0.001 0.0 0.0525" rpy="0.0 0.0 0.0"/>
-        <geometry>
-            <box size="0.002 0.025 0.105"/>
-        </geometry>
-    </visual>
-    <collision>
-        <origin xyz="-0.001 0.0 0.0525" rpy="0.0 0.0 0.0"/>
-        <geometry>
-            <box size="0.002 0.025 0.105"/>
-        </geometry>
-    </collision>
-    <visual>
-        <origin xyz="0.058 0.0 0.0525" rpy="0.0 0.0 0.0"/>
-        <geometry>
-            <box size="0.002 0.025 0.105"/>
-        </geometry>
-    </visual>
-    <collision>
-        <origin xyz="-0.001 0.0 0.0525" rpy="0.0 0.0 0.0"/>
+        <origin xyz="-0.001 0.000000001 0.0525" rpy="0.000000001 0.000000001 0.0000000001"/>
+        <geometry>
+            <box size="0.002 0.025 0.105"/>
+        </geometry>
+    </visual>
+    <collision>
+        <origin xyz="-0.001 0.000000001 0.0525" rpy="0.000000001 0.000000001 0.0000000001"/>
+        <geometry>
+            <box size="0.002 0.025 0.105"/>
+        </geometry>
+    </collision>
+    <visual>
+        <origin xyz="0.058 0.000000001 0.0525" rpy="0.000000001 0.000000001 0.0000000001"/>
+        <geometry>
+            <box size="0.002 0.025 0.105"/>
+        </geometry>
+    </visual>
+    <collision>
+        <origin xyz="-0.001 0.000000001 0.0525" rpy="0.000000001 0.000000001 0.0000000001"/>
         <geometry>
             <box size="0.002 0.025 0.105"/>
@@ -147,9 +147,9 @@
 <!--joint between bar 1 and bar 2-->
 <joint name="joint_3" type="revolute">
-    <origin xyz="-0.002 0.0 0.105" rpy="0.0 0.0 0.0"/>
+    <origin xyz="-0.002 0.000000001 0.105" rpy="0.000000001 0.000000001 0.0000000001"/>
     <parent link="bar1_link"/>
     <child link="bar2_link"/>
-    <axis xyz="-1.0 0.0 0.0"/>
-    <limit lower="-3.1415" upper="3.1415" effort="100" velocity="80"/>
+    <axis xyz="-1.0 0.000000001 0.0000000001"/>
+    <limit lower="-3.1415" upper="3.1415" effort="80" velocity="50"/>
 </joint>
 <!--bar 2 link-->
@@ -157,23 +157,23 @@
     <xacro:default_inertial mass="0.1"/>
     <visual>
-        <origin xyz="-0.001 0.0 0.049" rpy="0.0 0.0 0.0"/>
-        <geometry>
-            <box size="0.002 0.025 0.098"/>
-        </geometry>
-    </visual>
-    <collision>
-        <origin xyz="-0.001 0.0 0.049" rpy="0.0 0.0 0.0"/>
-        <geometry>
-            <box size="0.002 0.025 0.098"/>
-        </geometry>
-    </collision>
-    <visual>
-        <origin xyz="0.062 0.0 0.049" rpy="0.0 0.0 0.0"/>
-        <geometry>
-            <box size="0.002 0.025 0.098"/>
-        </geometry>
-    </visual>
-    <collision>
-        <origin xyz="0.062 0.0 0.049" rpy="0.0 0.0 0.0"/>
+        <origin xyz="-0.001 0.000000001 0.049" rpy="0.000000001 0.000000001 0.0000000001"/>
+        <geometry>
+            <box size="0.002 0.025 0.098"/>
+        </geometry>
+    </visual>
+    <collision>
+        <origin xyz="-0.001 0.000000001 0.049" rpy="0.000000001 0.000000001 0.0000000001"/>
+        <geometry>
+            <box size="0.002 0.025 0.098"/>
+        </geometry>
+    </collision>
+    <visual>
+        <origin xyz="0.062 0.000000001 0.049" rpy="0.000000001 0.000000001 0.0000000001"/>
+        <geometry>
+            <box size="0.002 0.025 0.098"/>
+        </geometry>
+    </visual>
+    <collision>
+        <origin xyz="0.062 0.000000001 0.049" rpy="0.000000001 0.000000001 0.0000000001"/>
         <geometry>
             <box size="0.002 0.025 0.098"/>
@@ -183,9 +183,9 @@
 <!--joint bar 2 motor 3-->
 <joint name="joint_4" type="revolute">
-    <origin xyz="0.002 0.0 0.098" rpy="0.0 0.0 0.0"/>
+    <origin xyz="0.002 0.000000001 0.098" rpy="0.000000001 0.000000001 0.0000000001"/>
     <parent link="bar2_link"/>
     <child link="motor3_link"/>
-    <axis xyz="-1.0 0.0 0.0"/>
-    <limit lower="-3.1415" upper="3.1415" effort="100" velocity="80"/>
+    <axis xyz="-1.0 0.000000001 0.0000000001"/>
+    <limit lower="-3.1415" upper="3.1415" effort="80" velocity="50"/>
 </joint>
 <!--motor 3 link-->
@@ -193,5 +193,5 @@
     <xacro:default_inertial mass="0.1"/>
     <visual>
-        <origin xyz="0.0285 0.01 0.0" rpy="0.0 0.0 0.0"/>
+        <origin xyz="0.0285 0.01 0.0000000001" rpy="0.000000001 0.000000001 0.0000000001"/>
         <geometry>
             <box size="0.056 0.06 0.025"/>
@@ -199,5 +199,5 @@
     </visual>
     <collision>
-        <origin xyz="0.0285 0.01 0.0" rpy="0.0 0.0 0.0"/>
+        <origin xyz="0.0285 0.01 0.0000000001" rpy="0.000000001 0.000000001 0.0000000001"/>
         <geometry>
             <box size="0.056 0.06 0.025"/>
@@ -207,5 +207,5 @@
 <!--motor 3 motor 4 joint-->
 <joint name="motor3_motor4_joint" type="fixed">
-    <origin xyz="0.0285 0.02 0.0125" rpy="0.0 0.0 0.0"/>
+    <origin xyz="0.0285 0.02 0.0125" rpy="0.000000001 0.000000001 0.0000000001"/>
     <parent link="motor3_link"/>
     <child link="motor4_link"/>
@@ -215,5 +215,5 @@
     <xacro:default_inertial mass="0.1"/>
     <visual>
-        <origin xyz="0.0 0.0 0.023" rpy="0.0 0.0 0.0"/>
+        <origin xyz="0.000000001 0.000000001 0.023" rpy="0.000000001 0.000000001 0.0000000001"/>
         <geometry>
             <box size="0.042 0.022 0.046"/>
@@ -221,5 +221,5 @@
     </visual>
     <collision>
-        <origin xyz="0.0 0.0 0.023" rpy="0.0 0.0 0.0"/>
+        <origin xyz="0.000000001 0.000000001 0.023" rpy="0.000000001 0.000000001 0.0000000001"/>
         <geometry>
             <box size="0.042 0.022 0.046"/>
@@ -229,9 +229,9 @@
 <!--Joint motor 4 ee link-->
 <joint name="joint_5" type="revolute">
-    <origin xyz="-0.01 0.0 0.046" rpy="0.0 0.0 0.0"/>
+    <origin xyz="-0.01 0.000000001 0.046" rpy="0.000000001 0.000000001 0.0000000001"/>
     <parent link="motor4_link"/>
     <child link="ee_link"/>
-    <axis xyz="0.0 0.0 1.0"/>
-    <limit lower="-3.1415" upper="3.1415" effort="100" velocity="80"/>
+    <axis xyz="0.000000001 0.000000001 1.0"/>
+    <limit lower="-3.1415" upper="3.1415" effort="80" velocity="50"/>
 </joint>
 <!-- ee link (end effector)-->
@@ -239,5 +239,5 @@
     <xacro:default_inertial mass="0.05"/>
     <visual>
-        <origin xyz="0.0 0.0 0.012" rpy="-1.57 0.0 0.0"/>
+        <origin xyz="0.000000001 0.000000001 0.012" rpy="-1.57 0.000000001 0.0000000001"/>
         <geometry>
             <cylinder radius="0.012" length="0.145"/>
@@ -245,5 +245,5 @@
     </visual>
     <collision>
-        <origin xyz="0.0 0.0 0.012" rpy="-1.57 0.0 0.0"/>
+        <origin xyz="0.000000001 0.000000001 0.012" rpy="-1.57 0.000000001 0.0000000001"/>
         <geometry>
             <cylinder radius="0.012" length="0.145"/>
