Commit message: Gazebo Simulation (gazebo.launch.py) + tested

File: arthrobot_ws/src/arthrobot_description/urdf/arthrobot.urdf.xacro (robot description, xacro)
@@ -3,6 +3,6 @@
     <!-- Useful XACRO Variables (Properties) -->
     <xacro:property name="PI" value="3.14159265359" />
-    <xacro:property name="effort" value="30.0000000001" />
-    <xacro:property name="velocity" value="10.0000000001" />
+    <xacro:property name="effort" value="30.0" />
+    <xacro:property name="velocity" value="10.0" />
     <!-- Useful Macros -->
     <xacro:macro name="default_inertial" params="mass">
@@ -10,6 +10,6 @@
             <origin xyz="0 0 0" rpy="0 0 0"/>
             <mass value="${mass}" />
-            <inertia ixx="1.0" ixy="0.0000000001" ixz="0.0000000001"
-                     iyy="1.0" iyz="0.0000000001"
+            <inertia ixx="1.0" ixy="0.0" ixz="0.0"
+                     iyy="1.0" iyz="0.0"
                      izz="1.0" />
         </inertial>
@@ -19,5 +19,5 @@
 <!--This is the joint that links the robot's base to the world frame -->
 <joint name="world_base_joint" type="fixed">
-    <origin xyz="0.000000001 0.000000001 0.0000000001" rpy="0.000000001 0.000000001 0.0000000001"/>
+    <origin xyz="0.0 0.0 0.0" rpy="0.0 0.0 0.0"/>
     <parent link="world"/>
     <child link="base_link"/>
@@ -27,5 +27,5 @@
     <xacro:default_inertial mass="2.0"/>
     <visual>
-        <origin xyz="0.000000001 0.000000001 0.0225" rpy="0.000000001 0.000000001 0.0000000001"/>
+        <origin xyz="0.0 0.0 0.0225" rpy="0.0 0.0 0.0"/>
         <geometry>
             <box size="0.19 0.16 0.045"/>
@@ -33,5 +33,5 @@
     </visual>
     <collision>
-        <origin xyz="0.000000001 0.000000001 0.00225" rpy="0.000000001 0.000000001 0.0000000001"/>
+        <origin xyz="0.0 0.0 0.00225" rpy="0.0 0.0 0.0"/>
         <geometry>
             <box size="0.19 0.16 0.045"/>
@@ -39,5 +39,5 @@
     </collision>
      <visual>
-        <origin xyz="-0.007 0.0085 0.063" rpy="0.000000001 0.000000001 0.0000000001"/>
+        <origin xyz="-0.007 0.0085 0.063" rpy="0.0 0.0 0.0"/>
         <geometry>
             <box size="0.07 0.06 0.036"/>
@@ -45,5 +45,5 @@
     </visual>
     <collision>
-        <origin xyz="-0.007 0.0085 0.063" rpy="0.000000001 0.000000001 0.0000000001"/>
+        <origin xyz="-0.007 0.0085 0.063" rpy="0.0 0.0 0.0"/>
         <geometry>
             <box size="0.07 0.06 0.036"/>
@@ -53,5 +53,5 @@
 <!-- Joint that attaches the base with motor 1-->
 <joint name="base_motor_link" type="fixed">
-    <origin xyz="-0.007 0.0085 0.081" rpy="0.000000001 0.000000001 0.0000000001"/>
+    <origin xyz="-0.007 0.0085 0.081" rpy="0.0 0.0 0.0"/>
     <parent link="base_link"/>
     <child link="motor1_link"/>
@@ -61,5 +61,5 @@
     <xacro:default_inertial mass="0.3"/>
     <visual>
-        <origin xyz="0.000000001 0.000000001 0.005" rpy="0.000000001 0.000000001 0.0000000001"/>
+        <origin xyz="0.0 0.0 0.005" rpy="0.0 0.0 0.0"/>
         <geometry>
             <box size="0.04 0.022 0.01"/>
@@ -67,5 +67,5 @@
     </visual>
     <collision>
-        <origin xyz="0.000000001 0.000000001 0.005" rpy="0.000000001 0.000000001 0.0000000001"/>
+        <origin xyz="0.0 0.0 0.005" rpy="0.0 0.0 0.0"/>
         <geometry>
             <box size="0.04 0.022 0.01"/>
@@ -73,5 +73,5 @@
     </collision>
     <visual>
-        <origin xyz="-0.01 0.000000001 0.014" rpy="0.000000001 0.000000001 0.0000000001"/>
+        <origin xyz="-0.01 0.0 0.014" rpy="0.0 0.0 0.0"/>
         <geometry>
             <cylinder radius="0.006" length="0.008"/>
@@ -79,5 +79,5 @@
     </visual>
     <collision>
-        <origin xyz="-0.01 0.000000001 0.004" rpy="0.000000001 0.000000001 0.0000000001"/>
+        <origin xyz="-0.01 0.0 0.004" rpy="0.0 0.0 0.0"/>
         <geometry>
             <cylinder radius="0.006" length="0.008"/>
@@ -87,8 +87,8 @@
 <!--Joint between motor 1 and motor 2-->
 <joint name="joint_1" type="revolute">
-    <origin xyz="-0.01 0.000000001 0.018" rpy="0.000000001 0.000000001 0.0000000001"/>
+    <origin xyz="-0.01 0.0 0.018" rpy="0.0 0.0 0.0"/>
     <parent link="motor1_link"/>
     <child link="motor2_link"/>
-    <axis xyz="0.000000001 0.000000001 1.0"/>
+    <axis xyz="0.0 0.0 1.0"/>
     <limit lower="-3.1415" upper="3.1415" effort="80" velocity="50"/>
 </joint>
@@ -97,5 +97,5 @@
     <xacro:default_inertial mass="0.2"/>
     <visual>
-        <origin xyz="0.000000001 0.01 0.0125" rpy="0.000000001 0.000000001 0.0000000001"/>
+        <origin xyz="0.0 0.01 0.0125" rpy="0.0 0.0 0.0"/>
         <geometry>
             <box size="0.057 0.06 0.025"/>
@@ -103,5 +103,5 @@
     </visual>
     <collision>
-        <origin xyz="0.000000001 0.01 0.0125" rpy="0.000000001 0.000000001 0.0000000001" />
+        <origin xyz="0.0 0.01 0.0125" rpy="0.0 0.0 0.0" />
         <geometry>
             <box size="0.057 0.06 0.025"/>
@@ -111,8 +111,8 @@
 <!--Joint between motor 2 and bar 1-->
 <joint name="joint_2" type="revolute">
-    <origin xyz="-0.0285 0.02 0.0125" rpy="0.000000001 0.000000001 0.0000000001"/>
+    <origin xyz="-0.0285 0.02 0.0125" rpy="0.0 0.0 0.0"/>
     <parent link="motor2_link"/>
     <child link="bar1_link"/>
-    <axis xyz="-1.0 0.000000001 0.0000000001"/>
+    <axis xyz="-1.0 0.0 0.0"/>
     <limit lower="-3.1415" upper="3.1415" effort="80" velocity="50"/>
 </joint>
@@ -121,23 +121,23 @@
     <xacro:default_inertial mass="0.1"/>
     <visual>
-        <origin xyz="-0.001 0.000000001 0.0525" rpy="0.000000001 0.000000001 0.0000000001"/>
-        <geometry>
-            <box size="0.002 0.025 0.105"/>
-        </geometry>
-    </visual>
-    <collision>
-        <origin xyz="-0.001 0.000000001 0.0525" rpy="0.000000001 0.000000001 0.0000000001"/>
-        <geometry>
-            <box size="0.002 0.025 0.105"/>
-        </geometry>
-    </collision>
-    <visual>
-        <origin xyz="0.058 0.000000001 0.0525" rpy="0.000000001 0.000000001 0.0000000001"/>
-        <geometry>
-            <box size="0.002 0.025 0.105"/>
-        </geometry>
-    </visual>
-    <collision>
-        <origin xyz="-0.001 0.000000001 0.0525" rpy="0.000000001 0.000000001 0.0000000001"/>
+        <origin xyz="-0.001 0.0 0.0525" rpy="0.0 0.0 0.0"/>
+        <geometry>
+            <box size="0.002 0.025 0.105"/>
+        </geometry>
+    </visual>
+    <collision>
+        <origin xyz="-0.001 0.0 0.0525" rpy="0.0 0.0 0.0"/>
+        <geometry>
+            <box size="0.002 0.025 0.105"/>
+        </geometry>
+    </collision>
+    <visual>
+        <origin xyz="0.058 0.0 0.0525" rpy="0.0 0.0 0.0"/>
+        <geometry>
+            <box size="0.002 0.025 0.105"/>
+        </geometry>
+    </visual>
+    <collision>
+        <origin xyz="-0.001 0.0 0.0525" rpy="0.0 0.0 0.0"/>
         <geometry>
             <box size="0.002 0.025 0.105"/>
@@ -147,8 +147,8 @@
 <!--joint between bar 1 and bar 2-->
 <joint name="joint_3" type="revolute">
-    <origin xyz="-0.002 0.000000001 0.105" rpy="0.000000001 0.000000001 0.0000000001"/>
+    <origin xyz="-0.002 0.0 0.105" rpy="0.0 0.0 0.0"/>
     <parent link="bar1_link"/>
     <child link="bar2_link"/>
-    <axis xyz="-1.0 0.000000001 0.0000000001"/>
+    <axis xyz="-1.0 0.0 0.0"/>
     <limit lower="-3.1415" upper="3.1415" effort="80" velocity="50"/>
 </joint>
@@ -157,23 +157,23 @@
     <xacro:default_inertial mass="0.1"/>
     <visual>
-        <origin xyz="-0.001 0.000000001 0.049" rpy="0.000000001 0.000000001 0.0000000001"/>
-        <geometry>
-            <box size="0.002 0.025 0.098"/>
-        </geometry>
-    </visual>
-    <collision>
-        <origin xyz="-0.001 0.000000001 0.049" rpy="0.000000001 0.000000001 0.0000000001"/>
-        <geometry>
-            <box size="0.002 0.025 0.098"/>
-        </geometry>
-    </collision>
-    <visual>
-        <origin xyz="0.062 0.000000001 0.049" rpy="0.000000001 0.000000001 0.0000000001"/>
-        <geometry>
-            <box size="0.002 0.025 0.098"/>
-        </geometry>
-    </visual>
-    <collision>
-        <origin xyz="0.062 0.000000001 0.049" rpy="0.000000001 0.000000001 0.0000000001"/>
+        <origin xyz="-0.001 0.0 0.049" rpy="0.0 0.0 0.0"/>
+        <geometry>
+            <box size="0.002 0.025 0.098"/>
+        </geometry>
+    </visual>
+    <collision>
+        <origin xyz="-0.001 0.0 0.049" rpy="0.0 0.0 0.0"/>
+        <geometry>
+            <box size="0.002 0.025 0.098"/>
+        </geometry>
+    </collision>
+    <visual>
+        <origin xyz="0.062 0.0 0.049" rpy="0.0 0.0 0.0"/>
+        <geometry>
+            <box size="0.002 0.025 0.098"/>
+        </geometry>
+    </visual>
+    <collision>
+        <origin xyz="0.062 0.0 0.049" rpy="0.0 0.0 0.0"/>
         <geometry>
             <box size="0.002 0.025 0.098"/>
@@ -183,8 +183,8 @@
 <!--joint bar 2 motor 3-->
 <joint name="joint_4" type="revolute">
-    <origin xyz="0.002 0.000000001 0.098" rpy="0.000000001 0.000000001 0.0000000001"/>
+    <origin xyz="0.002 0.0 0.098" rpy="0.0 0.0 0.0"/>
     <parent link="bar2_link"/>
     <child link="motor3_link"/>
-    <axis xyz="-1.0 0.000000001 0.0000000001"/>
+    <axis xyz="-1.0 0.0 0.0"/>
     <limit lower="-3.1415" upper="3.1415" effort="80" velocity="50"/>
 </joint>
@@ -193,5 +193,5 @@
     <xacro:default_inertial mass="0.1"/>
     <visual>
-        <origin xyz="0.0285 0.01 0.0000000001" rpy="0.000000001 0.000000001 0.0000000001"/>
+        <origin xyz="0.0285 0.01 0.0" rpy="0.0 0.0 0.0"/>
         <geometry>
             <box size="0.056 0.06 0.025"/>
@@ -199,5 +199,5 @@
     </visual>
     <collision>
-        <origin xyz="0.0285 0.01 0.0000000001" rpy="0.000000001 0.000000001 0.0000000001"/>
+        <origin xyz="0.0285 0.01 0.0" rpy="0.0 0.0 0.0"/>
         <geometry>
             <box size="0.056 0.06 0.025"/>
@@ -207,5 +207,5 @@
 <!--motor 3 motor 4 joint-->
 <joint name="motor3_motor4_joint" type="fixed">
-    <origin xyz="0.0285 0.02 0.0125" rpy="0.000000001 0.000000001 0.0000000001"/>
+    <origin xyz="0.0285 0.02 0.0125" rpy="0.0 0.0 0.0"/>
     <parent link="motor3_link"/>
     <child link="motor4_link"/>
@@ -215,5 +215,5 @@
     <xacro:default_inertial mass="0.1"/>
     <visual>
-        <origin xyz="0.000000001 0.000000001 0.023" rpy="0.000000001 0.000000001 0.0000000001"/>
+        <origin xyz="0.0 0.0 0.023" rpy="0.0 0.0 0.0"/>
         <geometry>
             <box size="0.042 0.022 0.046"/>
@@ -221,5 +221,5 @@
     </visual>
     <collision>
-        <origin xyz="0.000000001 0.000000001 0.023" rpy="0.000000001 0.000000001 0.0000000001"/>
+        <origin xyz="0.0 0.0 0.023" rpy="0.0 0.0 0.0"/>
         <geometry>
             <box size="0.042 0.022 0.046"/>
@@ -229,8 +229,8 @@
 <!--Joint motor 4 ee link-->
 <joint name="joint_5" type="revolute">
-    <origin xyz="-0.01 0.000000001 0.046" rpy="0.000000001 0.000000001 0.0000000001"/>
+    <origin xyz="-0.01 0.0 0.046" rpy="0.0 0.0 0.0"/>
     <parent link="motor4_link"/>
     <child link="ee_link"/>
-    <axis xyz="0.000000001 0.000000001 1.0"/>
+    <axis xyz="0.0 0.0 1.0"/>
     <limit lower="-3.1415" upper="3.1415" effort="80" velocity="50"/>
 </joint>
@@ -239,5 +239,5 @@
     <xacro:default_inertial mass="0.05"/>
     <visual>
-        <origin xyz="0.000000001 0.000000001 0.012" rpy="-1.57 0.000000001 0.0000000001"/>
+        <origin xyz="0.0 0.0 0.012" rpy="-1.57 0.0 0.0"/>
         <geometry>
             <cylinder radius="0.012" length="0.145"/>
@@ -245,5 +245,5 @@
     </visual>
     <collision>
-        <origin xyz="0.000000001 0.000000001 0.012" rpy="-1.57 0.000000001 0.0000000001"/>
+        <origin xyz="0.0 0.0 0.012" rpy="-1.57 0.0 0.0"/>
         <geometry>
             <cylinder radius="0.012" length="0.145"/>

Commit message: Configured ROS 2 Controller

File: arthrobot_ws/src/arthrobot_description/urdf/arthrobot.urdf.xacro (robot description, xacro)
@@ -1,4 +1,6 @@
 <?xml version="1.0"?>
 <robot xmlns:xacro="http://www.ros.org/wiki/xacro" name="arthrobot">
+    <xacro:include filename="$(find arthrobot_description)/urdf/arthrobot_gazebo.xacro"/>
+    <xacro:include filename="$(find arthrobot_description)/urdf/arthrobot_ros2_control.xacro"/>
     <!-- Useful XACRO Variables (Properties) -->
     <xacro:property name="PI" value="3.14159265359" />
@@ -15,4 +17,13 @@
         </inertial>
     </xacro:macro>
+    <xacro:macro name="default_transmission" params="number">
+        <transmission name="transmission_${number}">
+            <plugin>transmission_interface/SimpleTransmission</plugin>
+            <actuator name="motor_${number}" role="actuator1"/>
+            <joint name="joint_${number}" role="joint1">
+                <mechanical_reduction>1.0</mechanical_reduction>
+            </joint>
+        </transmission>
+    </xacro:macro>
 <!-- This is the first link: empty link specifying the world -->
 <link name="world"></link>
@@ -251,3 +262,8 @@
     </collision>
 </link>
+<xacro:default_transmission number="1"/>
+<xacro:default_transmission number="2"/>
+<xacro:default_transmission number="3"/>
+<xacro:default_transmission number="4"/>
+<xacro:default_transmission number="5"/>
 </robot>

Commit message: Cleaned up the repo

File: arthrobot_ws/src/arthrobot_description/urdf/arthrobot.urdf.xacro (robot description, xacro)
@@ -1,11 +1,42 @@
 <?xml version="1.0"?>
 <robot xmlns:xacro="http://www.ros.org/wiki/xacro" name="arthrobot">
-    <xacro:include filename="$(find arthrobot_description)/urdf/arthrobot_gazebo.xacro"/>
+    <!-- Include ros2_control Plugins -->
     <xacro:include filename="$(find arthrobot_description)/urdf/arthrobot_ros2_control.xacro"/>
-    <!-- Useful Variables -->
+    <!-- Useful XACRO Variables (Properties) -->
     <xacro:property name="PI" value="3.14159265359" />
-    <xacro:property name="effort" value="30.0" />
-    <xacro:property name="velocity" value="10.0" />
-    <!-- Useful Macros -->
+    <!-- Upper limits for joint efforts and velocities -->
+    <xacro:property name="link1_effort"        value="2"/>
+    <xacro:property name="link1_velocity"      value="1.0"/>
+    <xacro:property name="link2_effort"        value="2"/>
+    <xacro:property name="link2_velocity"      value="1.0"/>
+    <xacro:property name="link3_effort"        value="1"/>
+    <xacro:property name="link3_velocity"      value="1.0"/>
+    <xacro:property name="link4_effort"        value="1"/>
+    <xacro:property name="link4_velocity"      value="1.0"/>
+    <xacro:property name="link5_effort"       value="5"/>
+    <xacro:property name="link5_velocity"     value="1"/>
+    <xacro:property name="motor1_upper_limit"  value="${PI}"/>
+    <xacro:property name="motor1_lower_limit"  value="-${PI}"/>
+    <xacro:property name="motor2_upper_limit"  value="${PI}"/>
+    <xacro:property name="motor2_lower_limit"  value="-${PI}"/>
+    <xacro:property name="motor3_upper_limit"  value="${PI}"/>
+    <xacro:property name="motor3_lower_limit"  value="-${PI}"/>
+    <xacro:property name="motor4_upper_limit"  value="${PI}"/>
+    <xacro:property name="motor4_lower_limit"  value="-${PI}"/>
+    <xacro:property name="motor5_upper_limit"  value="${PI}"/>
+    <xacro:property name="motor5_lower_limit"  value="-${PI}"/>
+    <!-- Material Colors -->
+    <material name="black">
+        <color rgba="0.17 0.17 0.17 1.0"/>
+    </material>
+    <material name="gray">
+        <color rgba="0.6 0.6 0.6 1.0"/>
+    </material>
+    <material name="red">
+        <color rgba="0.9 0.05 0.05 1.0"/>
+    </material>
+    <material name="dark_gray">
+        <color rgba="0.2 0.2 0.2 1.0"/>
+    </material>
     <xacro:macro name="default_inertial" params="mass">
         <inertial>
@@ -17,17 +48,8 @@
         </inertial>
     </xacro:macro>
-    <xacro:macro name="default_transmission" params="number">
-        <transmission name="transmission_${number}">
-            <plugin>transmission_interface/SimpleTransmission</plugin>
-            <actuator name="motor_${number}" role="actuator1"/>
-            <joint name="joint_${number}" role="joint1">
-                <mechanical_reduction>1.0</mechanical_reduction>
-            </joint>
-        </transmission>
-    </xacro:macro>
 <!-- This is the first link: empty link specifying the world -->
 <link name="world"></link>
 <!--This is the joint that links the robot's base to the world frame -->
-<joint name="world_base_joint" type="fixed">
+<joint name="virtual_joint" type="fixed">
     <origin xyz="0.0 0.0 0.0" rpy="0.0 0.0 0.0"/>
     <parent link="world"/>
@@ -102,5 +124,6 @@
     <child link="motor2_link"/>
     <axis xyz="0.0 0.0 1.0"/>
-    <limit lower="-3.1415" upper="3.1415" effort="80" velocity="50"/>
+    <limit lower="${motor1_lower_limit}" upper="${motor1_upper_limit}"
+              effort="${link1_effort}" velocity="${link1_velocity}"/>
 </joint>
 <!--Motor 2 link-->
@@ -126,5 +149,6 @@
     <child link="bar1_link"/>
     <axis xyz="-1.0 0.0 0.0"/>
-    <limit lower="-3.1415" upper="3.1415" effort="80" velocity="50"/>
+    <limit lower="${motor2_lower_limit}" upper="${motor2_upper_limit}"
+              effort="${link2_effort}" velocity="${link2_velocity}"/>
 </joint>
 <!--bar 1 link-->
@@ -162,5 +186,6 @@
     <child link="bar2_link"/>
     <axis xyz="-1.0 0.0 0.0"/>
-    <limit lower="-3.1415" upper="3.1415" effort="80" velocity="50"/>
+    <limit lower="${motor3_lower_limit}" upper="${motor3_upper_limit}"
+              effort="${link3_effort}" velocity="${link3_velocity}"/>
 </joint>
 <!--bar 2 link-->
@@ -198,5 +223,6 @@
     <child link="motor3_link"/>
     <axis xyz="-1.0 0.0 0.0"/>
-    <limit lower="-3.1415" upper="3.1415" effort="80" velocity="50"/>
+    <limit lower="${motor4_lower_limit}" upper="${motor4_upper_limit}"
+              effort="${link4_effort}" velocity="${link4_velocity}"/>
 </joint>
 <!--motor 3 link-->
@@ -242,10 +268,11 @@
     <origin xyz="-0.01 0.0 0.046" rpy="0.0 0.0 0.0"/>
     <parent link="motor4_link"/>
-    <child link="ee_link"/>
+    <child link="motor5_link"/>
     <axis xyz="0.0 0.0 1.0"/>
-    <limit lower="-3.1415" upper="3.1415" effort="80" velocity="50"/>
-</joint>
-<!-- ee link (end effector)-->
-<link name="ee_link">
+    <limit lower="${motor5_lower_limit}" upper="${motor5_upper_limit}"
+              effort="${link5_effort}" velocity="${link5_velocity}"/>
+</joint>
+<!-- motor 5 link -->
+<link name="motor5_link">
     <xacro:default_inertial mass="0.05"/>
     <visual>
@@ -262,8 +289,3 @@
     </collision>
 </link>
-<xacro:default_transmission number="1"/>
-<xacro:default_transmission number="2"/>
-<xacro:default_transmission number="3"/>
-<xacro:default_transmission number="4"/>
-<xacro:default_transmission number="5"/>
 </robot>

File: arthrobot_ws/src/arthrobot_description/urdf/arthrobot_ros2_control.xacro (robot description, xacro)
@@ -3,40 +3,57 @@
     <ros2_control name="RobotSystem" type="system">
         <xacro:property name="PI" value="3.14159265359" />
-        <!-- ros2_control Gazebo -->
+        <xacro:property name="motor1_upper_limit"  value="${PI}"/>
+        <xacro:property name="motor1_lower_limit"  value="-${PI}"/>
+        <xacro:property name="motor2_upper_limit"  value="${PI}"/>
+        <xacro:property name="motor2_lower_limit"  value="-${PI}"/>
+        <xacro:property name="motor3_upper_limit"  value="${PI}"/>
+        <xacro:property name="motor3_lower_limit"  value="-${PI}"/>
+        <xacro:property name="motor4_upper_limit"  value="${PI}"/>
+        <xacro:property name="motor4_lower_limit"  value="-${PI}"/>
+        <xacro:property name="motor5_upper_limit"  value="${PI}"/>
+        <xacro:property name="motor5_lower_limit"  value="-${PI}"/>
+        <!-- Custom Hardware Interface -->
         <hardware>
-            <plugin>gazebo_ros2_control/GazeboSystem</plugin>
+            <plugin>byrot_arm_controller/ArthrobotHardwareInterface</plugin>
         </hardware>
+        <!-- BYROT's Arm -->
         <joint name="joint_1">
+            <param name="initial_position">0.0</param>
             <command_interface name="position">
-            <param name="min">-${PI}</param>
-            <param name="max">${PI}</param>
+                <param name="min">motor1_lower_limit</param>
+                <param name="max">motor1_upper_limit</param>
             </command_interface>
             <state_interface name="position"/>
         </joint>
         <joint name="joint_2">
+            <param name="initial_position">0.0</param>
             <command_interface name="position">
-            <param name="min">-${PI}</param>
-            <param name="max">${PI}</param>
+                <param name="min">motor2_lower_limit</param>
+                <param name="max">motor2_upper_limit</param>
             </command_interface>
             <state_interface name="position"/>
         </joint>
         <joint name="joint_3">
+            <param name="initial_position">0.0</param>
             <command_interface name="position">
-            <param name="min">-${PI}</param>
-            <param name="max">${PI}</param>
+                <param name="min">motor3_lower_limit</param>
+                <param name="max">motor3_upper_limit</param>
             </command_interface>
             <state_interface name="position"/>
         </joint>
         <joint name="joint_4">
+            <param name="initial_position">0.0</param>
             <command_interface name="position">
-            <param name="min">-${PI}</param>
-            <param name="max">${PI}</param>
+                <param name="min">motor4_lower_limit</param>
+                <param name="max">motor4_upper_limit</param>
             </command_interface>
             <state_interface name="position"/>
         </joint>
+        <!-- BYROT's gripper -->
         <joint name="joint_5">
+            <param name="initial_position">0.0</param>
             <command_interface name="position">
-            <param name="min">-${PI}</param>
-            <param name="max">${PI}</param>
+                <param name="min">motor4_lower_limit</param>
+                <param name="max">motor4_upper_limit</param>
             </command_interface>
             <state_interface name="position"/>
