Commit message: Updated the end-effector to be more realistic, matching Arthrobot's structure

File: arthrobot_ws/src/arthrobot_description/urdf/arthrobot.urdf.xacro (robot description, xacro)
@@ -277,5 +277,5 @@
     <xacro:default_inertial mass="0.05"/>
     <visual>
-        <origin xyz="0.0 0.0 0.012" rpy="-1.57 0.0 0.0"/>
+        <origin xyz="0.0 0.0725 0.012" rpy="-1.57 0.0 0.0"/>
         <geometry>
             <cylinder radius="0.012" length="0.145"/>
@@ -283,5 +283,5 @@
     </visual>
     <collision>
-        <origin xyz="0.0 0.0 0.012" rpy="-1.57 0.0 0.0"/>
+        <origin xyz="0.0 0.0725 0.012" rpy="-1.57 0.0 0.0"/>
         <geometry>
             <cylinder radius="0.012" length="0.145"/>
@@ -289,3 +289,47 @@
     </collision>
 </link>
+<!-- End effector support joint-->
+<joint name="joint_ee_support" type="fixed">
+    <origin xyz="0.0 0.145 0.012" rpy="0.0 0.0 0.0"/>
+    <parent link="motor5_link"/>
+    <child link="ee_link_support"/>
+</joint>
+<!-- End effector support link -->
+<link name="ee_link_support">
+    <xacro:default_inertial mass="0.05"/>
+    <visual>
+        <origin xyz="0.0 0.0 0.0" rpy="0.0 0.0 0.0"/>
+        <geometry>
+            <cylinder radius="0.012" length="0.012"/>
+        </geometry>
+    </visual>
+    <collision>
+        <origin xyz="0.0 0.0 0.0" rpy="0.0 0.0 0.0"/>
+        <geometry>
+            <cylinder radius="0.012" length="0.012"/>
+        </geometry>
+    </collision>
+</link>
+<!-- End effector joint-->
+<joint name="joint_ee" type="fixed">
+    <origin xyz="0.0 0.0 0.0" rpy="0.0 0.0 0.0"/>
+    <parent link="ee_link_support"/>
+    <child link="ee_link"/>
+</joint>
+<!-- End effector link -->
+<link name="ee_link">
+    <xacro:default_inertial mass="0.05"/>
+    <visual>
+        <origin xyz="0.0 0.0 0.0" rpy="0.0 0.0 0.0"/>
+        <geometry>
+            <cylinder radius="0.012" length="0.012"/>
+        </geometry>
+    </visual>
+    <collision>
+        <origin xyz="0.0 0.0 0.0" rpy="0.0 0.0 0.0"/>
+        <geometry>
+            <cylinder radius="0.012" length="0.012"/>
+        </geometry>
+    </collision>
+</link>
 </robot>

Commit message: The interface with MG996R motors from ROS 2 was set (Using the PCA9685 I2C PWM Driver)

File: arthrobot_ws/src/arthrobot_description/urdf/arthrobot.urdf.xacro (robot description, xacro)
@@ -16,14 +16,15 @@
     <xacro:property name="link5_effort"       value="5"/>
     <xacro:property name="link5_velocity"     value="1"/>
-    <xacro:property name="motor1_upper_limit"  value="${PI}"/>
-    <xacro:property name="motor1_lower_limit"  value="-${PI}"/>
-    <xacro:property name="motor2_upper_limit"  value="${PI}"/>
-    <xacro:property name="motor2_lower_limit"  value="-${PI}"/>
-    <xacro:property name="motor3_upper_limit"  value="${PI}"/>
-    <xacro:property name="motor3_lower_limit"  value="-${PI}"/>
-    <xacro:property name="motor4_upper_limit"  value="${PI}"/>
-    <xacro:property name="motor4_lower_limit"  value="-${PI}"/>
-    <xacro:property name="motor5_upper_limit"  value="${PI}"/>
-    <xacro:property name="motor5_lower_limit"  value="-${PI}"/>
+    <xacro:property name="PI" value="3.14159265359" />
+    <xacro:property name="motor1_upper_limit"  value="${PI/2}"/>
+    <xacro:property name="motor1_lower_limit"  value="-${PI/2}"/>
+    <xacro:property name="motor2_upper_limit"  value="${PI/2}"/>
+    <xacro:property name="motor2_lower_limit"  value="-${PI/2}"/>
+    <xacro:property name="motor3_upper_limit"  value="${PI/2}"/>
+    <xacro:property name="motor3_lower_limit"  value="-${PI/2}"/>
+    <xacro:property name="motor4_upper_limit"  value="${PI/2}"/>
+    <xacro:property name="motor4_lower_limit"  value="-${PI/2}"/>
+    <xacro:property name="motor5_upper_limit"  value="${PI/2}"/>
+    <xacro:property name="motor5_lower_limit"  value="-${PI/2}"/>
     <!-- Material Colors -->
     <material name="black">

File: arthrobot_ws/src/arthrobot_description/urdf/arthrobot_ros2_control.xacro (robot description, xacro)
@@ -3,14 +3,14 @@
     <ros2_control name="RobotSystem" type="system">
         <xacro:property name="PI" value="3.14159265359" />
-        <xacro:property name="motor1_upper_limit"  value="${PI}"/>
-        <xacro:property name="motor1_lower_limit"  value="-${PI}"/>
-        <xacro:property name="motor2_upper_limit"  value="${PI}"/>
-        <xacro:property name="motor2_lower_limit"  value="-${PI}"/>
-        <xacro:property name="motor3_upper_limit"  value="${PI}"/>
-        <xacro:property name="motor3_lower_limit"  value="-${PI}"/>
-        <xacro:property name="motor4_upper_limit"  value="${PI}"/>
-        <xacro:property name="motor4_lower_limit"  value="-${PI}"/>
-        <xacro:property name="motor5_upper_limit"  value="${PI}"/>
-        <xacro:property name="motor5_lower_limit"  value="-${PI}"/>
+        <xacro:property name="motor1_upper_limit"  value="${PI/2}"/>
+        <xacro:property name="motor1_lower_limit"  value="-${PI/2}"/>
+        <xacro:property name="motor2_upper_limit"  value="${PI/2}"/>
+        <xacro:property name="motor2_lower_limit"  value="-${PI/2}"/>
+        <xacro:property name="motor3_upper_limit"  value="${PI/2}"/>
+        <xacro:property name="motor3_lower_limit"  value="-${PI/2}"/>
+        <xacro:property name="motor4_upper_limit"  value="${PI/2}"/>
+        <xacro:property name="motor4_lower_limit"  value="-${PI/2}"/>
+        <xacro:property name="motor5_upper_limit"  value="${PI/2}"/>
+        <xacro:property name="motor5_lower_limit"  value="-${PI/2}"/>
         <!-- Custom Hardware Interface -->
         <hardware>
