Commit message: real-time control GUI improved and improved the servoing params

File: arthrobot_ws/src/arthrobot_description/urdf/arthrobot.urdf.xacro (robot description, xacro)
@@ -129,4 +129,19 @@
         </visual>
     </link>
+    <!-- Extra joint for the interactive marker -->
+    <joint name="gripper_support_joint" type="fixed">
+        <origin xyz="0.0 0.1 0.0" rpy="0.0 0.0 0.0"/>
+        <parent link="palm_link"/>
+        <child link="gripper_support"/>
+    </joint>
+    <link name="gripper_support">
+    <visual>
+        <!-- small visual to mark the new link -->
+        <origin xyz="0 0 0" rpy="0 0 0"/>
+        <geometry>
+            <box size="0.005 0.005 0.005"/>
+        </geometry>
+        </visual>
+    </link>
     <joint name="gripper_joint" type="revolute">
         <origin xyz="0.003 0.0385 0.0035" rpy="0.0 0.0 0.0"/>

Commit message: Integrated the ArthroBot gripper in the MoveIt planning pipeline

File: arthrobot_ws/src/arthrobot_description/urdf/arthrobot.urdf.xacro (robot description, xacro)
@@ -149,5 +149,5 @@
         <child link="right_finger_base_link"/>
         <axis xyz="0.0 0.0 -1.0"/>
-        <limit lower="${gripper_lower_limit}" upper="${shoulder_upper_limit}" effort="2.0" velocity="2.0"/>
+        <limit lower="${gripper_lower_limit}" upper="${gripper_upper_limit}" effort="2.0" velocity="2.0"/>
     </joint>
     <link name="right_finger_base_link">
@@ -165,5 +165,5 @@
         <child link="left_finger_base_link"/>
         <axis xyz="0.0 0.0 -1.0"/>
-        <limit lower="0.0" upper="1.5708" effort="2.0" velocity="2.0"/>
+        <limit lower="-1.5708" upper="0.0" effort="2.0" velocity="2.0"/>
         <mimic joint="gripper_joint" multiplier="-1" offset="0"/>
     </joint>
@@ -182,5 +182,5 @@
         <child link="right_finger_link"/>
         <axis xyz="0.0 0.0 -1.0"/>
-        <limit lower="0.0" upper="1.5708" effort="2.0" velocity="2.0"/>
+        <limit lower="0.0" upper="1.9" effort="2.0" velocity="2.0"/>
         <mimic joint="gripper_joint" multiplier="1.2" offset="0"/>
     </joint>
@@ -199,5 +199,5 @@
         <child link="left_finger_link"/>
         <axis xyz="0.0 0.0 -1.0"/>
-        <limit lower="0.0" upper="1.5708" effort="2.0" velocity="2.0"/>
+        <limit lower="-1.9" upper="0.0" effort="2.0" velocity="2.0"/>
         <mimic joint="palm_left_finger_base_joint" multiplier="1.2" offset="0"/>
     </joint>
@@ -233,5 +233,5 @@
         <child link="right_fingertip_link"/>
         <axis xyz="0.0 0.0 -1.0"/>
-        <limit lower="0.0" upper="1.5708" effort="2.0" velocity="2.0"/>
+        <limit lower="-1.5708" upper="0.0" effort="2.0" velocity="2.0"/>
         <mimic joint="gripper_joint" multiplier="-1" offset="0"/>
     </joint>

Commit message: Added collision object + IK approximation + Controller integration

File: arthrobot_ws/src/arthrobot_description/urdf/arthrobot.urdf.xacro (robot description, xacro)
@@ -64,4 +64,10 @@
         <material name="gray"/>
         </visual>
+        <collision>
+        <geometry>
+            <mesh filename="package://arthrobot_description/meshes/waist_link.stl" scale="0.001 0.001 0.001"/>
+        </geometry>
+        <origin rpy="0.0 0.0 0.0" xyz="0.0 0.0 0.0"/>
+        </collision>
     </link>
     <joint name="shoulder_joint" type="revolute">
@@ -80,4 +86,10 @@
         <material name="gray"/>
         </visual>
+        <collision>
+        <geometry>
+            <mesh filename="package://arthrobot_description/meshes/shoulder_link.stl" scale="0.001 0.001 0.001"/>
+        </geometry>
+        <origin rpy="0.0 0.0 0.0" xyz="0.0 0.0 0.0"/>
+        </collision>
     </link>
     <joint name="forearm_joint" type="revolute">
@@ -96,4 +108,10 @@
         <material name="gray"/>
         </visual>
+        <collision>
+        <geometry>
+            <mesh filename="package://arthrobot_description/meshes/forearm_link.stl" scale="0.001 0.001 0.001"/>
+        </geometry>
+        <origin rpy="0.0 0.0 0.0" xyz="0.0 0.0 0.0"/>
+        </collision>
     </link>
     <joint name="wrist_joint" type="revolute">
@@ -112,4 +130,10 @@
         <material name="gray"/>
         </visual>
+        <collision>
+        <geometry>
+            <mesh filename="package://arthrobot_description/meshes/wrist_link.stl" scale="0.001 0.001 0.001"/>
+        </geometry>
+        <origin rpy="0.0 0.0 0.0" xyz="0.0 0.0 0.0"/>
+        </collision>
     </link>
     <joint name="palm_joint" type="revolute">
@@ -128,4 +152,10 @@
         <material name="gray"/>
         </visual>
+        <collision>
+        <geometry>
+            <mesh filename="package://arthrobot_description/meshes/palm_link.stl" scale="0.001 0.001 0.001"/>
+        </geometry>
+        <origin rpy="0.0 0.0 0.0" xyz="0.0 0.0 0.0"/>
+        </collision>
     </link>
     <!-- Extra joint for the interactive marker -->
@@ -227,4 +257,10 @@
         <material name="gray"/>
         </visual>
+        <collision>
+        <geometry>
+            <mesh filename="package://arthrobot_description/meshes/left_fingertip_link.stl" scale="0.001 0.001 0.001"/>
+        </geometry>
+        <origin rpy="0.0 0.0 0.0" xyz="0.0 0.0 0.0"/>
+        </collision>
     </link>
     <joint name="right_fingertip_joint" type="revolute">
@@ -244,4 +280,10 @@
         <material name="gray"/>
         </visual>
+        <collision>
+        <geometry>
+            <mesh filename="package://arthrobot_description/meshes/right_fingertip_link.stl" scale="0.001 0.001 0.001"/>
+        </geometry>
+        <origin rpy="0.0 0.0 0.0" xyz="0.0 0.0 0.0"/>
+        </collision>
     </link>
 </robot>

Commit message: Ready for demo commit

File: arthrobot_ws/src/arthrobot_description/urdf/arthrobot.urdf.xacro (robot description, xacro)
@@ -161,5 +161,5 @@
     <!-- Extra joint for the interactive marker -->
     <joint name="gripper_support_joint" type="fixed">
-        <origin xyz="0.0 0.1 0.0" rpy="0.0 0.0 0.0"/>
+        <origin xyz="-0.005 0.1 0.0" rpy="0.0 0.0 0.0"/>
         <parent link="palm_link"/>
         <child link="gripper_support"/>
